File: USBCPD_PCB/_autosave-USBCPD_PCB.kicad_sch (KiCad schematic)
At the start: 64 parts, among them IC1 TMCS1108A3BQDRQ1, IC2 UCC27282QDRQ1, IC3 UCC27282QDRQ1, IC4 BAJ2CC0FP-E2, J1 TB002-500-02BE, J2 TB002-500-02BE, Q1 SIR584DP-T1-RE3, Q2 SIR584DP-T1-RE3, Q3 SIR584DP-T1-RE3, Q4 SIR584DP-T1-RE3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

Commit message: libs added, routing finalized, fixed issues
copied libs into folder, wrong wiring fixed, added test pads and silkscreen
Parts:
- gave numbers to parts that had none: 4
Changed lines of the file:
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@@
   (symbol (lib_id "Connector:TestPoint") (at 171.45 261.62 180) (unit 1)
     (in_bom yes) (on_board yes) (dnp no) (fields_autoplaced)
-    (property "Reference" "TP?" (at 173.99 264.287 0)
+    (property "Reference" "TP7" (at 173.99 264.287 0)
       (effects (font (size 1.27 1.27)) (justify right))
     )
@@
       (project "USBCPD_PCB"
         (path "/d348c750-b8a4-4ea0-a85d-ac4257fd8477"
-          (reference "TP?") (unit 1)
+          (reference "TP7") (unit 1)
         )
       )
@@
   (symbol (lib_id "Connector:TestPoint") (at 171.45 227.33 0) (unit 1)
     (in_bom yes) (on_board yes) (dnp no) (fields_autoplaced)
-    (property "Reference" "TP?" (at 173.99 223.393 0)
+    (property "Reference" "TP6" (at 173.99 223.393 0)
       (effects (font (size 1.27 1.27)) (justify left))
     )
@@
       (project "USBCPD_PCB"
         (path "/d348c750-b8a4-4ea0-a85d-ac4257fd8477"
-          (reference "TP?") (unit 1)
+          (reference "TP6") (unit 1)
         )
       )
@@
   (symbol (lib_id "Connector:TestPoint") (at 281.94 261.62 180) (unit 1)
     (in_bom yes) (on_board yes) (dnp no) (fields_autoplaced)
-    (property "Reference" "TP?" (at 284.48 264.287 0)
+    (property "Reference" "TP10" (at 284.48 264.287 0)
       (effects (font (size 1.27 1.27)) (justify right))
     )
@@
       (project "USBCPD_PCB"
         (path "/d348c750-b8a4-4ea0-a85d-ac4257fd8477"
-          (reference "TP?") (unit 1)
+          (reference "TP10") (unit 1)
         )
       )
@@
   (symbol (lib_id "Connector:TestPoint") (at 281.94 226.06 0) (unit 1)
     (in_bom yes) (on_board yes) (dnp no) (fields_autoplaced)
-    (property "Reference" "TP?" (at 284.48 222.123 0)
+    (property "Reference" "TP9" (at 284.48 222.123 0)
       (effects (font (size 1.27 1.27)) (justify left))
     )
@@
       (project "USBCPD_PCB"
         (path "/d348c750-b8a4-4ea0-a85d-ac4257fd8477"
-          (reference "TP?") (unit 1)
+          (reference "TP9") (unit 1)
         )
       )
