File: USBCPD_PCB/USBCPD_PCB.kicad_pcb (KiCad board)
At the start: 2 copper layers, 69.6 x 51.3 mm, 65 parts, among them IC1 TMCS1108A3BQDRQ1, IC2 UCC27282QDRQ1, IC3 UCC27282QDRQ1, IC4 BAJ2CC0FP-E2, J1 TB002-500-02BE, J2 TB002-500-02BE, Q1 SIR584DP-T1-RE3, Q2 SIR584DP-T1-RE3, Q3 SIR584DP-T1-RE3, Q4 SIR584DP-T1-RE3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

Commit message: schematic rewire changes & hotfixes
Parts:
- R10: value 2.8K -> 16k
- R9: value 900R -> 1k
Connections:
- R1 pad 1: PA9_PWM -> PB12_PWM
- R13 pad 2: PA10_ADC_Vout -> PC2_ADC_Vout
- R14 pad 1: PA10_ADC_Vout -> PC2_ADC_Vout
- R2 pad 1: PA8_PWM -> PB13_PWM
- R5 pad 2: PB3_ADC_Iout -> PC3_ADC_Iout
- R7 pad 1: PB13_PWM -> PB15_PWM
- U1 pad CN10_16: PB12_LED -> PB12_PWM
- U1 pad CN10_21: PA9_PWM -> unconnected-(U1B-PA9-PadCN10_21)
- U1 pad CN10_23: PA8_PWM -> PA8_LED
- U1 pad CN10_26: unconnected-(U1B-PB15-PadCN10_26) -> PB15_PWM
- U1 pad CN10_31: PB3_ADC_Iout -> unconnected-(U1B-PB3-PadCN10_31)
- U1 pad CN10_33: PA10_ADC_Vout -> unconnected-(U1B-PA10-PadCN10_33)
- U1 pad CN7_35: unconnected-(U1A-PC2-PadCN7_35) -> PC2_ADC_Vout
- U1 pad CN7_37: unconnected-(U1A-PC3-PadCN7_37) -> PC3_ADC_Iout
Routing:
- net PA8_PWM: track 51.9 -> 0.00 mm
- net PA9_PWM: track 51.1 -> 0.00 mm
- net PB14_PWM: track 49.0 -> 0.00 mm, vias 1 -> 0
- net PA10_ADC_Vout: track 45.7 -> 0.00 mm
- net PB13_PWM: track 40.8 -> 0.00 mm, vias 1 -> 0
- net PB3_ADC_Iout: track 35.5 -> 0.00 mm, vias 1 -> 0
- net PB12_LED: track 18.5 -> 0.00 mm
