File: USBCPD_PCB/USBCPD_PCB.kicad_sch (KiCad schematic)
At the start: 64 parts, among them IC1 TMCS1108A3BQDRQ1, IC2 UCC27282QDRQ1, IC3 UCC27282QDRQ1, IC4 BAJ2CC0FP-E2, J1 TB002-500-02BE, J2 TB002-500-02BE, Q1 SIR584DP-T1-RE3, Q2 SIR584DP-T1-RE3, Q3 SIR584DP-T1-RE3, Q4 SIR584DP-T1-RE3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

Commit message: save
Parts:
- removed unit 5 of U1
- removed unit 4 of U1
- removed unit 3 of U1
- removed unit 6 of U1
- gave numbers to parts that had none: 4
Connections:
- no-connect marks 85 -> 54

Commit message: tons of errors
Parts:
- R10: value 2.8K -> 16k
- R9: value 900R -> 1k
Other:
- note added: "high R, due to losses"
Changed lines of the file:
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@@
     (effects (font (size 1.27 1.27)) (justify right bottom))
   )
+  (text "high R, due to losses" (at 350.52 213.36 0)
+    (effects (font (size 1.27 1.27)) (justify left bottom))
+  )
   (text "3.2V 20mA Blue" (at 332.74 226.695 0)
     (effects (font (size 1.27 1.27)) (justify right bottom))
@@
       (effects (font (size 1.27 1.27)) (justify left))
     )
-    (property "Value" "900R" (at 342.9 208.915 0)
+    (property "Value" "1k" (at 342.9 208.915 0)
       (effects (font (size 1.27 1.27)) (justify left))
     )
@@
       (effects (font (size 1.27 1.27)) (justify left))
     )
-    (property "Value" "2.8K" (at 372.11 210.185 0)
+    (property "Value" "16k" (at 372.11 210.185 0)
       (effects (font (size 1.27 1.27)) (justify left))
     )

Commit message: schematic rewire changes & hotfixes
Connections:
- net PB12_LED: no longer U1.CN10_16 (PB12)
- net PB13_PWM: now also R2.1; no longer R7.1
- net PC2_ADC_Vout: now reaches U1.CN7_35 (PC2)
- net PC2_ADC_Vout: now also R13.2, R14.1
- net PC3_ADC_Iout: now reaches U1.CN7_37 (PC3)
- net PC3_ADC_Iout: now also R5.2
- net PB15_PWM: now reaches U1.CN10_26 (PB15)
- net PB15_PWM: now also R7.1
- removed net PA10_ADC_Vout: R13.2, R14.1, U1.CN10_33 (PA10)
- net PA8_PWM renamed PA8_LED
- net PA8_LED: no longer R2.1
- net PA9_PWM: no longer names the net of U1.CN10_21 (PA9)
- net PA9_PWM: no longer R1.1
- net PB3_ADC_Iout: no longer names the net of U1.CN10_31 (PB3)
- net PB3_ADC_Iout: no longer R5.2
- new net PB12_PWM: R1.1, U1.CN10_16 (PB12)

Commit message: save
Connections:
- net PB12_PWM: now also R2.1; no longer R1.1
- net PB13_PWM: now also R1.1; no longer R2.1
- net PB14_PWM: now also R7.1; no longer R6.1
- net PB15_PWM: now also R6.1; no longer R7.1
